Commit message: Update A3.2 hand models and control workflows; add right P01-P04 motions

File: assets/hands/TsenseI_hand_v3_2_withid/source_20_outputs/TsenseI_hand_left_v3_2_withid.urdf (robot description, URDF)
Before this commit: robot TsenseI_hand_v3_2_withid_left, 22 links, 21 joints
Links:
- link Left_hand_palm_link: mass None -> 0.017000000000000001; geometry collision mesh filename=../meshes/left/left_hand_palm_support__P0090.STL scale=1 1 1; visual mesh filename=../meshes/left/left_hand_palm_support__P0090.STL scale=1 1 1
- link base_link: mass None -> 0.14999999999999999; geometry collision mesh filename=../meshes/left/left_hand_base_electronics__P0216.STL scale=1 1 1; collision mesh filename=../meshes/left/left_hand_base_electronics__P0230.STL scale=1 1 1
- link left_hand_index_DIP_link: mass None -> 0.014999999999999999; geometry collision mesh filename=../meshes/left/left_hand_index_tip_bearing__P0240.STL scale=1 1 1; collision mesh filename=../meshes/left/left_hand_index_tip_bearing__P0243.STL scale=1 1 1
- link left_hand_index_MCP_link: mass None -> 0.029999999999999999; geometry collision mesh filename=../meshes/left/left_hand_index_swing_bearing__P0267.STL scale=1 1 1; collision mesh filename=../meshes/left/left_hand_index_swing_electronics__P0270.STL scale=1 1 1
- link left_hand_index_PIP_link: mass None -> 0.040000000000000001; geometry collision mesh filename=../meshes/left/left_hand_index_DIP_bearing__P0245.STL scale=1 1 1; collision mesh filename=../meshes/left/left_hand_index_DIP_electronics_motor_stator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 scale=1 1 1
- link left_hand_index_swing_link: mass None -> 0.070000000000000007; geometry collision mesh filename=../meshes/left/left_hand_index_PIP_bearing__P0246.STL scale=1 1 1; collision mesh filename=../meshes/left/left_hand_index_PIP_electronics_motor_stator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 scale=1 1 1
- link left_hand_mid_DIP_link: mass None -> 0.014999999999999999; geometry collision mesh filename=../meshes/left/left_hand_mid_tip_bearing__STD004_P0240.STL scale=1 1 1; collision mesh filename=../meshes/left/left_hand_mid_tip_bearing__STD004_P0243.STL scale=1 1 1
- link left_hand_mid_MCP_link: mass None -> 0.029999999999999999; geometry collision mesh filename=../meshes/left/left_hand_mid_swing_bearing__P0314.STL scale=1 1 1; collision mesh filename=../meshes/left/left_hand_mid_swing_electronics__P0316.STL scale=1 1 1
- link left_hand_mid_PIP_link: mass None -> 0.040000000000000001; geometry collision mesh filename=../meshes/left/left_hand_mid_DIP_bearing__STD004_P0245.STL scale=1 1 1; collision mesh filename=../meshes/left/left_hand_mid_DIP_electronics_motor_stator__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 scale=1 1 1
- link left_hand_mid_swing_link: mass None -> 0.070000000000000007; geometry collision mesh filename=../meshes/left/left_hand_mid_PIP_bearing__P0329.STL scale=1 1 1; collision mesh filename=../meshes/left/left_hand_mid_PIP_electronics_motor_stator__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 scale=1 1 1
- link left_hand_pinky_DIP_link: mass None -> 0.014999999999999999; geometry collision mesh filename=../meshes/left/left_hand_pinky_tip_bearing__P0415.STL scale=1 1 1; collision mesh filename=../meshes/left/left_hand_pinky_tip_bearing__P0417.STL scale=1 1 1
- link left_hand_pinky_MCP_link: mass None -> 0.029999999999999999; geometry collision mesh filename=../meshes/left/left_hand_pinky_swing_bearing__P0435.STL scale=1 1 1; collision mesh filename=../meshes/left/left_hand_pinky_swing_electronics__P0422.STL scale=1 1 1
- link left_hand_pinky_PIP_link: mass None -> 0.040000000000000001; geometry collision mesh filename=../meshes/left/left_hand_pinky_DIP_bearing__P0387.STL scale=1 1 1; collision mesh filename=../meshes/left/left_hand_pinky_DIP_bearing__P0389.STL scale=1 1 1
- link left_hand_pinky_swing_link: mass None -> 0.070000000000000007; geometry collision mesh filename=../meshes/left/left_hand_pinky_PIP_electronics_motor_stator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 scale=1 1 1; collision mesh filename=../meshes/left/left_hand_pinky_PIP_fastener__P0388.STL scale=1 1 1
- link left_hand_ring_DIP_link: mass None -> 0.014999999999999999; geometry collision mesh filename=../meshes/left/left_hand_ring_tip_bearing__P0000.STL scale=1 1 1; collision mesh filename=../meshes/left/left_hand_ring_tip_bearing__P0012.STL scale=1 1 1
- link left_hand_ring_MCP_link: mass None -> 0.029999999999999999; geometry collision mesh filename=../meshes/left/left_hand_ring_swing_bearing__P0029.STL scale=1 1 1; collision mesh filename=../meshes/left/left_hand_ring_swing_electronics__P0035.STL scale=1 1 1
- link left_hand_ring_PIP_link: mass None -> 0.040000000000000001; geometry collision mesh filename=../meshes/left/left_hand_ring_DIP_bearing__P0015.STL scale=1 1 1; collision mesh filename=../meshes/left/left_hand_ring_DIP_electronics_motor_stator_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 scale=1 1 1
- link left_hand_ring_swing_link: mass None -> 0.070000000000000007; geometry collision mesh filename=../meshes/left/left_hand_ring_PIP_bearing__P0016.STL scale=1 1 1; collision mesh filename=../meshes/left/left_hand_ring_PIP_electronics_motor_stator_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 scale=1 1 1
- link left_hand_thumb_MCP_link: mass None -> 0.040000000000000001; geometry collision mesh filename=../meshes/left/left_hand_thumb_MCP_fastener__P0367.STL scale=1 1 1; collision mesh filename=../meshes/left/left_hand_thumb_MCP_fastener__P0377.STL scale=1 1 1
- link left_hand_thumb_PIP_link: mass None -> 0.014999999999999999; geometry collision mesh filename=../meshes/left/left_hand_thumb_tip_bearing__P0382.STL scale=1 1 1; collision mesh filename=../meshes/left/left_hand_thumb_tip_bearing__P0384.STL scale=1 1 1
- link left_hand_thumb_rota_block_link: mass None -> 0.035000000000000003; geometry collision mesh filename=../meshes/left/left_hand_thumb_rotation2_fastener__P0335.STL scale=1 1 1; collision mesh filename=../meshes/left/left_hand_thumb_rotation2_fastener__P0337.STL scale=1 1 1
- link left_hand_thumb_rotaback_link2: mass None -> 0.074999999999999997; geometry collision mesh filename=../meshes/left/left_hand_thumb_MCP_electronics_motor_stator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 scale=1 1 1; collision mesh filename=../meshes/left/left_hand_thumb_MCP_fastener__P0360.STL scale=1 1 1
Joints:
- joint Left_hand_palm_joint: axis 0 0 0 -> (none); origin xyz=0.023699999999999999 0.0064999999999999997 0.044138006984399999 rpy=0 0 0 -> xyz=0.023699999999999999 0.0064999999999999997 0.044138006984399999 rpy=-0 0 -0
- joint left_hand_index_DIP_joint: limit lower=0.0 upper=1.5707963267948966 effort=1.0 velocity=1.0 -> lower=0.0 upper=1.57 effort=1.0 velocity=1.0; origin xyz=-0.0053114137261469213 0.025846448194837987 -0.0045110466755889644 rpy=-2.7755575615628914e-17 0 0.12903783821920917 -> xyz=-0.005311413721869232 0.025846448194579805 -1.1900203045200897e-15 rpy=-2.7755575615628914e-17 0 0.12903783821920919
- joint left_hand_index_MCP_joint: limit lower=0.0 upper=1.5707963267948966 effort=1.0 velocity=1.0 -> lower=0.0 upper=1.57 effort=1.0 velocity=1.0; origin xyz=0.027106823283284235 -0.026576387592038783 0.087815835680192231 rpy=1.4508509931644693 0.42625833852372441 3.084615774699254 -> xyz=0.027099703634998501 -0.027567214335181868 0.087707234999650913 rpy=1.4508509931644693 0.42625833852372441 3.084615774699254
- joint left_hand_index_PIP_joint: limit lower=0.0 upper=1.5707963267948966 effort=1.0 velocity=1.0 -> lower=0.0 upper=1.57 effort=1.0 velocity=1.0; origin xyz=0.041023546156784746 3.4694469519536142e-18 -0.026999999999999597 rpy=1.5707963267948963 -1.1967399807955119 3.1077098616583827 -> xyz=0.041999999999999843 -6.9388939039072284e-18 -0.026999999999998192 rpy=1.5707963267948972 -1.1967399807954855 3.141592653589786
- joint left_hand_index_swing_joint: origin xyz=0.01819644753826806 0.019340354107076171 -0.00099999999999282954 rpy=1.5707963267948957 -0.033882791931409972 2.0005586058915599 -> xyz=0.018196447538264333 0.019340354107076393 -3.2139486642566995e-06 rpy=1.5707963267948974 -6.4392935428259079e-15 2.0005586058915856
- joint left_hand_mid_DIP_joint: limit lower=0.0 upper=1.5707963267948966 effort=1.0 velocity=1.0 -> lower=0.0 upper=1.57 effort=1.0 velocity=1.0; origin xyz=-0.0053114137261472405 0.025846448194837821 -0.0017315940115265904 rpy=-5.5511151231257827e-17 0 0.12903783821923204 -> xyz=-0.0053114137218693014 0.02584644819457986 -5.9934696094998685e-16 rpy=-2.7755575615628914e-17 0 0.12903783821921641
- joint left_hand_mid_MCP_joint: limit lower=0.0 upper=1.5707963267948966 effort=1.0 velocity=1.0 -> lower=0.0 upper=1.57 effort=1.0 velocity=1.0; origin xyz=0.02719999953837687 -0.00049999877805580509 0.088138007230611604 rpy=1.5707963267948968 0.4297622790966602 -3.1415926535897896 -> xyz=0.027099703634997883 -0.0015860674645024192 0.088138007230611604 rpy=1.5707963267948961 0.42976227909668507 3.1344499886106498
- joint left_hand_mid_PIP_joint: limit lower=0.0 upper=1.5707963267948966 effort=1.0 velocity=1.0 -> lower=0.0 upper=1.57 effort=1.0 velocity=1.0; origin xyz=0.041023559408067872 2.1684043449710089e-19 -0.026019547123553179 rpy=1.5707963267948974 -1.1967399807954628 -3.1077095759704942 -> xyz=0.041999999999999524 2.1684043449710089e-19 -0.025300000000000357 rpy=1.5707963267948983 -1.196739980795503 -3.1415926535897833
- joint left_hand_mid_swing_joint: origin xyz=0.017305157670401285 0.018931832119254491 -0.00099998783788761165 rpy=1.570796326794897 0.033883077619299762 2.0005586058915852 -> xyz=0.016651037339347238 0.018632041099237523 -3.2139486486977478e-06 rpy=1.570796326794897 1.021405182655144e-14 2.0005586058915852
- joint left_hand_pinky_DIP_joint: limit lower=0.0 upper=1.5707963267948966 effort=1.0 velocity=1.0 -> lower=0.0 upper=1.57 effort=1.0 velocity=1.0; origin xyz=-0.0063815055464910009 0.025204810461647131 -0.006034842938728309 rpy=-0.0062711979857275647 0.025075123623853113 -0.00012198116402359176 -> xyz=-0.0063032454065007973 0.025224375205066263 0.00020675515638993863 rpy=-0.0062711979857275543 0.025075123623853113 -0.00012198116402324438
- joint left_hand_pinky_MCP_joint: limit lower=0.0 upper=1.5707963267948966 effort=1.0 velocity=1.0 -> lower=0.0 upper=1.57 effort=1.0 velocity=1.0; origin xyz=0.0271068232832797 0.044704606014039389 0.070250121398440751 rpy=1.7043559433280713 0.42725082875541354 -3.0931711956586163 -> xyz=0.027099703634997516 0.043715192884881314 0.07037092455483579 rpy=1.7043559433280713 0.42725082875541376 -3.0931711956586163
- joint left_hand_pinky_PIP_joint: limit lower=0.0 upper=1.5707963267948966 effort=1.0 velocity=1.0 -> lower=0.0 upper=1.57 effort=1.0 velocity=1.0; origin xyz=0.038626320568843936 0 -0.02181000000000018 rpy=1.5707963267948963 -1.3258211702687228 3.0606963287343296 -> xyz=0.039500000000000451 0 -0.021809999999998733 rpy=1.5707963267948983 -1.3258211702686955 3.1415926535897452
- joint left_hand_pinky_swing_joint: origin xyz=0.018196447538267484 0.019340354107076102 -0.0010000000000004935 rpy=1.5707963267948957 -0.080896324855458834 2.0005586058915581 -> xyz=0.01819644753826722 0.019340354107075734 -3.2139486648014026e-06 rpy=1.570796326794897 -4.2188474935755949e-14 2.0005586058915821
- joint left_hand_ring_DIP_joint: limit lower=0.0 upper=1.5707963267948966 effort=1.0 velocity=1.0 -> lower=0.0 upper=1.57 effort=1.0 velocity=1.0; origin xyz=-0.0053114137258253313 0.025846448194971533 -0.0045110466755893131 rpy=-2.7755575615628914e-17 0 0.12903783821922418 -> xyz=-0.0053114137218728263 0.025846448194579971 -1.8496055381733711e-12 rpy=-2.7755575615628914e-17 0 0.12903783821922268
- joint left_hand_ring_MCP_joint: limit lower=0.0 upper=1.5707963267948966 effort=1.0 velocity=1.0 -> lower=0.0 upper=1.57 effort=1.0 velocity=1.0; origin xyz=0.027106823283282962 0.023481417630913871 0.080906629963767754 rpy=1.6667660125609922 0.42864098926106586 -3.1087726476133142 -> xyz=0.027099703634997717 0.022488449981419661 0.080993503376345019 rpy=1.6667660125609913 0.42864098926109384 -3.1087726476133133
- joint left_hand_ring_PIP_joint: limit lower=0.0 upper=1.5707963267948966 effort=1.0 velocity=1.0 -> lower=0.0 upper=1.57 effort=1.0 velocity=1.0; origin xyz=0.04102354615678494 -1.7347234759768071e-18 -0.026999999999998935 rpy=1.570796326794895 -1.1967399807954981 3.107709861658404 -> xyz=0.041999999999998067 3.4694469519536142e-18 -0.026999999999994938 rpy=1.570796326794897 -1.1967399807954719 -3.14159265358979
- joint left_hand_ring_swing_joint: origin xyz=0.018196447538267047 0.019340354107075949 -0.00099999999999785677 rpy=1.5707963267948961 -0.03388279193139021 2.0005586058915599 -> xyz=0.018196447538263112 0.019340354107076241 -3.2139486561156422e-06 rpy=1.5707963267948979 2.4424906541753444e-15 2.0005586058916132
- joint left_hand_thumb_MCP_joint: limit lower=0.0 upper=1.5707963267948966 effort=1.0 velocity=1.0 -> lower=0.0 upper=1.57 effort=1.0 velocity=1.0; origin xyz=0.051777369955726356 -1.3877787807814457e-17 0.0054157007354755024 rpy=0.5275107839615536 -0.9084965891297635 -2.3106248516321068 -> xyz=0.051668942592601144 0 -0.0052920750176667572 rpy=0.52751078396112183 -0.90849658912994835 -2.2879591616094781
- joint left_hand_thumb_PIP_joint: limit lower=0.0 upper=1.5707963267948966 effort=1.0 velocity=1.0 -> lower=0.0 upper=1.57 effort=1.0 velocity=1.0; origin xyz=-0.0053114137218719798 0.025846448194579846 -0.0045110466755894085 rpy=1.6792123247455493e-15 2.4424906541753444e-15 0.12903783821924114 -> xyz=-0.0053114137218506358 0.025846448194589706 -2.0539125955565396e-15 rpy=3.8857805861880479e-16 -4.2188474935755949e-15 0.1290378382195399
- joint left_hand_thumb_rota_block_joint: origin xyz=0.020095209458105473 -0.018319894388608274 0.034425784821471982 rpy=0.409849353962845 0.035990946425296544 -1.099842689237515 -> xyz=0.024488440509375025 -0.01869491074294765 0.036060974991322353 rpy=0.35982319468221313 0.20381117386131797 -1.5108048438524189
- joint left_hand_thumb_rotaback_joint2: axis 0 0 -1 -> -0 -0 -1; limit lower=0.0 upper=1.7400000000000002 effort=1.0 velocity=1.0 -> lower=0.0 upper=1.74 effort=1.0 velocity=1.0; origin xyz=0.025906534761571742 -3.4694469519536142e-18 -0.010516065096279111 rpy=1.5707963267949003 -1.1774916255348222 -0.55582153100282139 -> xyz=0.022315626236229048 -1.3877787807814457e-17 -0.0123000641755272 rpy=1.5707963267948892 -1.5247423161228992 -0.16657232709293579
