Commit message: Update A3.2 hand models and control workflows; add right P01-P04 motions

File: assets/hands/TsenseI_hand_v3_2_withid/urdf/TsenseI_hand_right_v3_2_withid.urdf (robot description, URDF)
Before this commit: robot TsenseI_hand_v3_2_withid_right, 22 links, 21 joints
Links:
- link Right_hand_palm_link: mass None -> 0.017000000000000001; geometry collision mesh filename=../mjcf/collision_meshes/right_Right_hand_palm_link.stl; visual mesh filename=../meshes/right/right_hand_palm_support__P0090.STL scale=1 1 1
- link base_link: mass None -> 0.14999999999999999; geometry collision mesh filename=../mjcf/collision_meshes/right_base_link.stl; visual mesh filename=../meshes/right/right_hand_base_electronics__P0216.STL scale=1 1 1
- link right_hand_index_DIP_link: mass None -> 0.014999999999999999; geometry collision mesh filename=../mjcf/collision_meshes/right_right_hand_index_DIP_link.stl; visual mesh filename=../meshes/right/right_hand_index_tip_bearing__P0240.STL scale=1 1 1
- link right_hand_index_MCP_link: mass None -> 0.029999999999999999; geometry collision mesh filename=../mjcf/collision_meshes/right_right_hand_index_MCP_link.stl; visual mesh filename=../meshes/right/right_hand_index_swing_bearing__P0267.STL scale=1 1 1
- link right_hand_index_PIP_link: mass None -> 0.040000000000000001; geometry collision mesh filename=../mjcf/collision_meshes/right_right_hand_index_PIP_link.stl; visual mesh filename=../meshes/right/right_hand_index_DIP_bearing__P0245.STL scale=1 1 1
- link right_hand_index_swing_link: mass None -> 0.070000000000000007; geometry collision mesh filename=../mjcf/collision_meshes/right_right_hand_index_swing_link.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; visual mesh filename=../meshes/right/right_hand_index_PIP_bearing__P0246.STL scale=1 1 1
- link right_hand_mid_DIP_link: mass None -> 0.014999999999999999; geometry collision mesh filename=../mjcf/collision_meshes/right_right_hand_mid_DIP_link.stl; visual mesh filename=../meshes/right/right_hand_mid_tip_bearing__STD004_P0240.STL scale=1 1 1
- link right_hand_mid_MCP_link: mass None -> 0.029999999999999999; geometry collision mesh filename=../mjcf/collision_meshes/right_right_hand_mid_MCP_link.stl; visual mesh filename=../meshes/right/right_hand_mid_swing_bearing__P0314.STL scale=1 1 1
- link right_hand_mid_PIP_link: mass None -> 0.040000000000000001; geometry collision mesh filename=../mjcf/collision_meshes/right_right_hand_mid_PIP_link.stl; visual mesh filename=../meshes/right/right_hand_mid_DIP_bearing__STD004_P0245.STL scale=1 1 1
- link right_hand_mid_swing_link: mass None -> 0.070000000000000007; geometry collision mesh filename=../mjcf/collision_meshes/right_right_hand_mid_swing_link.stl; visual mesh filename=../meshes/right/right_hand_mid_PIP_bearing__P0329.STL scale=1 1 1
- link right_hand_pinky_DIP_link: mass None -> 0.014999999999999999; geometry collision mesh filename=../mjcf/collision_meshes/right_right_hand_pinky_DIP_link.stl; visual mesh filename=../meshes/right/right_hand_pinky_tip_bearing__P0415.STL scale=1 1 1
- link right_hand_pinky_MCP_link: mass None -> 0.029999999999999999; geometry collision mesh filename=../mjcf/collision_meshes/right_right_hand_pinky_MCP_link.stl; visual mesh filename=../meshes/right/right_hand_pinky_swing_bearing__P0435.STL scale=1 1 1
- link right_hand_pinky_PIP_link: mass None -> 0.040000000000000001; geometry collision mesh filename=../mjcf/collision_meshes/right_right_hand_pinky_PIP_link.stl; visual mesh filename=../meshes/right/right_hand_pinky_DIP_bearing__P0387.STL scale=1 1 1
- link right_hand_pinky_swing_link: mass None -> 0.070000000000000007; geometry collision mesh filename=../mjcf/collision_meshes/right_right_hand_pinky_swing_link.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; visual mesh filename=../meshes/right/right_hand_pinky_PIP_electronics_motor_stat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 scale=1 1 1
- link right_hand_ring_DIP_link: mass None -> 0.014999999999999999; geometry collision mesh filename=../mjcf/collision_meshes/right_right_hand_ring_DIP_link.stl; visual mesh filename=../meshes/right/right_hand_ring_tip_bearing__P0000.STL scale=1 1 1
- link right_hand_ring_MCP_link: mass None -> 0.029999999999999999; geometry collision mesh filename=../mjcf/collision_meshes/right_right_hand_ring_MCP_link.stl; visual mesh filename=../meshes/right/right_hand_ring_swing_bearing__P0029.STL scale=1 1 1
- link right_hand_ring_PIP_link: mass None -> 0.040000000000000001; geometry collision mesh filename=../mjcf/collision_meshes/right_right_hand_ring_PIP_link.stl; visual mesh filename=../meshes/right/right_hand_ring_DIP_bearing__P0015.STL scale=1 1 1
- link right_hand_ring_swing_link: mass None -> 0.070000000000000007; geometry collision mesh filename=../mjcf/collision_meshes/right_right_hand_ring_swing_link.s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; visual mesh filename=../meshes/right/right_hand_ring_PIP_bearing__P0016.STL scale=1 1 1
- link right_hand_thumb_MCP_link: mass None -> 0.040000000000000001; geometry collision mesh filename=../mjcf/collision_meshes/right_right_hand_thumb_MCP_link.stl; visual mesh filename=../meshes/right/right_hand_thumb_MCP_fastener__P0367.STL scale=1 1 1
- link right_hand_thumb_PIP_link: mass None -> 0.014999999999999999; geometry collision mesh filename=../mjcf/collision_meshes/right_right_hand_thumb_PIP_link.stl; visual mesh filename=../meshes/right/right_hand_thumb_tip_bearing__P0382.STL scale=1 1 1
- link right_hand_thumb_rota_block_link: mass None -> 0.035000000000000003; geometry collision mesh filename=../mjcf/collision_meshes/right_right_hand_thumb_rota_block_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; visual mesh filename=../meshes/right/right_hand_thumb_rotation2_fastener__P0335.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 scale=1 1 1
- link right_hand_thumb_rotaback_link2: mass None -> 0.074999999999999997; geometry collision mesh filename=../mjcf/collision_meshes/right_right_hand_thumb_rotaback_li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; visual mesh filename=../meshes/right/right_hand_thumb_MCP_electronics_motor_stat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 scale=1 1 1
Joints:
- joint Right_hand_palm_joint: axis 0 0 0 -> (none); origin xyz=0.0237 -0.0065 0.0441380069844 rpy=0 0 0 -> xyz=0.023699999999999999 0.0015000000000000005 0.044138006984399999 rpy=0 0 0
- joint right_hand_index_DIP_joint: origin xyz=-0.00531141372614692 -0.025846448194838 -0.00451104667558896 rpy=0 0 -0.129037838219209 -> xyz=-0.005311413721869232 -0.025846448194579805 -1.1900203045200897e-15 rpy=2.7755575615628914e-17 0 -0.12903783821920919
- joint right_hand_index_MCP_joint: origin xyz=0.0271068232832842 0.0265763875920388 0.0878158356801922 rpy=-1.45085099316447 0.426258338523724 -3.08461577469925 -> xyz=0.027099703634998501 0.035567214335181868 0.087707234999650913 rpy=-1.4508509931644693 0.42625833852372441 -3.084615774699254
- joint right_hand_index_PIP_joint: origin xyz=0.0410235461567847 0 -0.0269999999999996 rpy=-1.5707963267949 -1.19673998079551 -3.10770986165838 -> xyz=0.041999999999999843 6.9388939039072284e-18 -0.026999999999998192 rpy=-1.5707963267948972 -1.1967399807954855 -3.141592653589786
- joint right_hand_index_swing_joint: origin xyz=0.0181964475382681 -0.0193403541070762 -0.00099999999999283 rpy=-1.5707963267949 -0.03388279193141 -2.00055860589156 -> xyz=0.018196447538264333 -0.019340354107076393 -3.2139486642566995e-06 rpy=-1.5707963267948974 -6.4392935428259079e-15 -2.0005586058915856
- joint right_hand_mid_DIP_joint: origin xyz=-0.00531141372614724 -0.0258464481948378 -0.00173159401152659 rpy=0 0 -0.129037838219232 -> xyz=-0.0053114137218693014 -0.02584644819457986 -5.9934696094998685e-16 rpy=2.7755575615628914e-17 0 -0.12903783821921641
- joint right_hand_mid_MCP_joint: origin xyz=0.0271999995383769 0.000499998778055805 0.0881380072306116 rpy=-1.5707963267949 0.42976227909666 3.14159265358979 -> xyz=0.027099703634997883 0.0095860674645024194 0.088138007230611604 rpy=-1.5707963267948961 0.42976227909668507 -3.1344499886106498
- joint right_hand_mid_PIP_joint: origin xyz=0.0410235594080679 0 -0.0260195471235532 rpy=-1.5707963267949 -1.19673998079546 3.10770957597049 -> xyz=0.041999999999999524 -2.1684043449710089e-19 -0.025300000000000357 rpy=-1.5707963267948983 -1.196739980795503 3.1415926535897833
- joint right_hand_mid_swing_joint: origin xyz=0.0173051576704013 -0.0189318321192545 -0.000999987837887612 rpy=-1.5707963267949 0.0338830776192998 -2.00055860589159 -> xyz=0.016651037339347238 -0.018632041099237523 -3.2139486486977478e-06 rpy=-1.570796326794897 1.021405182655144e-14 -2.0005586058915852
- joint right_hand_pinky_DIP_joint: origin xyz=-0.006381505546491 -0.0252048104616471 -0.00603484293872831 rpy=0.00627119798572756 0.0250751236238531 0.000121981164023592 -> xyz=-0.0063032454065007973 -0.025224375205066263 0.00020675515638993863 rpy=0.0062711979857275543 0.025075123623853113 0.00012198116402324438
- joint right_hand_pinky_MCP_joint: origin xyz=0.0271068232832797 -0.0447046060140394 0.0702501213984408 rpy=-1.70435594332807 0.427250828755414 3.09317119565862 -> xyz=0.027099703634997516 -0.035715192884881314 0.07037092455483579 rpy=-1.7043559433280713 0.42725082875541376 3.0931711956586163
- joint right_hand_pinky_PIP_joint: origin xyz=0.0386263205688439 0 -0.0218100000000002 rpy=-1.5707963267949 -1.32582117026872 -3.06069632873433 -> xyz=0.039500000000000451 0 -0.021809999999998733 rpy=-1.5707963267948983 -1.3258211702686955 -3.1415926535897452
- joint right_hand_pinky_swing_joint: origin xyz=0.0181964475382675 -0.0193403541070761 -0.00100000000000049 rpy=-1.5707963267949 -0.0808963248554588 -2.00055860589156 -> xyz=0.01819644753826722 -0.019340354107075734 -3.2139486648014026e-06 rpy=-1.570796326794897 -4.2188474935755949e-14 -2.0005586058915821
- joint right_hand_ring_DIP_joint: origin xyz=-0.00531141372582533 -0.0258464481949715 -0.00451104667558931 rpy=0 0 -0.129037838219224 -> xyz=-0.0053114137218728263 -0.025846448194579971 -1.8496055381733711e-12 rpy=2.7755575615628914e-17 0 -0.12903783821922268
- joint right_hand_ring_MCP_joint: origin xyz=0.027106823283283 -0.0234814176309139 0.0809066299637678 rpy=-1.66676601256099 0.428640989261066 3.10877264761331 -> xyz=0.027099703634997717 -0.014488449981419661 0.080993503376345019 rpy=-1.6667660125609913 0.42864098926109384 3.1087726476133133
- joint right_hand_ring_PIP_joint: origin xyz=0.0410235461567849 0 -0.0269999999999989 rpy=-1.5707963267949 -1.1967399807955 -3.1077098616584 -> xyz=0.041999999999998067 -3.4694469519536142e-18 -0.026999999999994938 rpy=-1.570796326794897 -1.1967399807954719 3.14159265358979
- joint right_hand_ring_swing_joint: origin xyz=0.018196447538267 -0.0193403541070759 -0.000999999999997857 rpy=-1.5707963267949 -0.0338827919313902 -2.00055860589156 -> xyz=0.018196447538263112 -0.019340354107076241 -3.2139486561156422e-06 rpy=-1.5707963267948979 2.4424906541753444e-15 -2.0005586058916132
- joint right_hand_thumb_MCP_joint: origin xyz=0.0517773699557264 0 0.0054157007354755 rpy=-0.527510783961554 -0.908496589129763 2.31062485163211 -> xyz=0.051668942592601144 0 -0.0052920750176667572 rpy=-0.52751078396112183 -0.90849658912994835 2.2879591616094781
- joint right_hand_thumb_PIP_joint: origin xyz=-0.00531141372187198 -0.0258464481945798 -0.00451104667558941 rpy=-1.67921232474555e-15 2.44249065417534e-15 -0.129037838219241 -> xyz=-0.0053114137218506358 -0.025846448194589706 -2.0539125955565396e-15 rpy=-3.8857805861880479e-16 -4.2188474935755949e-15 -0.1290378382195399
- joint right_hand_thumb_rota_block_joint: origin xyz=0.0200952094581055 0.0183198943886083 0.034425784821472 rpy=-0.409849353962845 0.0359909464252965 1.09984268923752 -> xyz=0.024488440509375025 0.02669491074294765 0.036060974991322353 rpy=-0.35982319468221313 0.20381117386131797 1.5108048438524189
- joint right_hand_thumb_rotaback_joint2: axis 0 0 1 -> -0.0 -0.0 1.0; origin xyz=0.0259065347615717 0 -0.0105160650962791 rpy=-1.5707963267949 -1.17749162553482 0.555821531002821 -> xyz=0.022315626236229048 1.3877787807814457e-17 -0.0123000641755272 rpy=-1.5707963267948892 -1.5247423161228992 0.16657232709293579
