Commit message: Update Ubuntu hand control project and exclude archives

File: assets/hands/TsenseI_hand_v3_2/urdf/TsenseI_hand_left_v3_2.urdf (robot description, URDF)
Before this commit: robot TsenseI_hand_v3_2_left, 22 links, 21 joints
Joints:
- joint left_hand_index_MCP_joint: limit lower=0.005 upper=1.3 effort=0 velocity=0 -> lower=0.005 upper=1.565 effort=0 velocity=0
- joint left_hand_index_swing_joint: axis 1 0 0 -> -1 -0 -0; limit lower=0.0 upper=0.7 effort=0 velocity=0 -> lower=-0.35 upper=0.35 effort=0 velocity=0; origin xyz=-0.0134 0 0.01 rpy=-0.35000000000000003 0 0 -> xyz=-0.0134 0 0.01 rpy=-5.5511151231257839e-17 0 0
- joint left_hand_mid_MCP_joint: limit lower=0.005 upper=1.3 effort=0 velocity=0 -> lower=0.005 upper=1.565 effort=0 velocity=0
- joint left_hand_mid_swing_joint: axis 1 0 0 -> -1 -0 -0; limit lower=0.0 upper=0.7 effort=0 velocity=0 -> lower=-0.35 upper=0.35 effort=0 velocity=0; origin xyz=-0.014875 0 0.01 rpy=-0.35000000000000003 0 0 -> xyz=-0.014875 0 0.01 rpy=-5.5511151231257839e-17 0 0
- joint left_hand_pinky_MCP_joint: limit lower=0.005 upper=1.3 effort=0 velocity=0 -> lower=0.005 upper=1.565 effort=0 velocity=0
- joint left_hand_pinky_swing_joint: axis 1 0 0 -> -1 -0 -0; limit lower=0.0 upper=0.7 effort=0 velocity=0 -> lower=-0.35 upper=0.35 effort=0 velocity=0; origin xyz=-0.016925 0 0.01 rpy=-0.35000000000000003 0 0 -> xyz=-0.016925 0 0.01 rpy=-5.5511151231257839e-17 0 0
- joint left_hand_ring_MCP_joint: limit lower=0.005 upper=1.3 effort=0 velocity=0 -> lower=0.005 upper=1.565 effort=0 velocity=0
- joint left_hand_ring_swing_joint: axis 1 0 0 -> -1 -0 -0; limit lower=0.0 upper=0.7 effort=0 velocity=0 -> lower=-0.35 upper=0.35 effort=0 velocity=0; origin xyz=-0.0149 0 0.01 rpy=-0.35000000000000003 0 0 -> xyz=-0.0149 0 0.01 rpy=-5.5511151231257839e-17 0 0
- joint left_hand_thumb_MCP_joint: limit lower=0.005 upper=1.3 effort=0 velocity=0 -> lower=0.005 upper=1.565 effort=0 velocity=0
- joint left_hand_thumb_rotaback_joint2: origin xyz=-0.0091878 -0.019669 -0.00042716 rpy=-0.25042009379455915 0 -0.18193999999999999 -> xyz=-0.0091878 -0.019669 -0.00042716 rpy=2.7755575615628914e-17 0 -0.18194000000000002

File: assets/hands/TsenseI_hand_v3_2/urdf/TsenseI_hand_right_v3_2.urdf (robot description, URDF)
Before this commit: robot TsenseI_hand_v3_2_right, 22 links, 21 joints
Joints:
- joint right_hand_index_MCP_joint: limit lower=0.005 upper=1.3 effort=0 velocity=0 -> lower=0.005 upper=1.565 effort=0 velocity=0
- joint right_hand_index_swing_joint: axis 1 0 0 -> -1 -0 -0; limit lower=0.0 upper=0.7 effort=0 velocity=0 -> lower=-0.35 upper=0.35 effort=0 velocity=0; origin xyz=0.0134 0 0.01 rpy=-0.35000000000000003 0 0 -> xyz=0.0134 0 0.01 rpy=-5.5511151231257839e-17 0 0
- joint right_hand_mid_MCP_joint: limit lower=0.005 upper=1.3 effort=0 velocity=0 -> lower=0.005 upper=1.565 effort=0 velocity=0
- joint right_hand_mid_swing_joint: axis 1 0 0 -> -1 -0 -0; limit lower=0.0 upper=0.7 effort=0 velocity=0 -> lower=-0.35 upper=0.35 effort=0 velocity=0; origin xyz=0.014875 0 0.01 rpy=-0.35000000000000003 0 0 -> xyz=0.014875 0 0.01 rpy=-5.5511151231257839e-17 0 0
- joint right_hand_pinky_MCP_joint: limit lower=0.005 upper=1.3 effort=0 velocity=0 -> lower=0.005 upper=1.565 effort=0 velocity=0
- joint right_hand_pinky_swing_joint: axis 1 0 0 -> -1 -0 -0; limit lower=0.0 upper=0.7 effort=0 velocity=0 -> lower=-0.35 upper=0.35 effort=0 velocity=0; origin xyz=0.016925 0 0.01 rpy=-0.35000000000000003 0 0 -> xyz=0.016925 0 0.01 rpy=-5.5511151231257839e-17 0 0
- joint right_hand_ring_MCP_joint: limit lower=0.005 upper=1.3 effort=0 velocity=0 -> lower=0.005 upper=1.565 effort=0 velocity=0
- joint right_hand_ring_swing_joint: axis 1 0 0 -> -1 -0 -0; limit lower=0.0 upper=0.7 effort=0 velocity=0 -> lower=-0.35 upper=0.35 effort=0 velocity=0; origin xyz=0.0149 0 0.01 rpy=-0.35000000000000003 0 0 -> xyz=0.0149 0 0.01 rpy=-5.5511151231257839e-17 0 0
- joint right_hand_thumb_MCP_joint: limit lower=0.005 upper=1.3 effort=0 velocity=0 -> lower=0.005 upper=1.565 effort=0 velocity=0
- joint right_hand_thumb_rotaback_joint2: origin xyz=0.0091878 -0.019669 -0.00042716 rpy=-0.25042009379455915 0 0.18193999999999999 -> xyz=0.0091878 -0.019669 -0.00042716 rpy=2.7755575615628914e-17 0 0.18194000000000002

File: assets/hands/TsenseI_hand_v3_2_withid/urdf/TsenseI_hand_left_v3_2_withid.urdf (robot description, URDF)
Before this commit: robot TsenseI_hand_v3_2_withid_left, 22 links, 21 joints
Links:
- link Left_hand_palm_link: mass 0.017 -> None; geometry collision mesh filename=../mjcf/collision_meshes/left_Left_hand_palm_link.stl; visual mesh filename=../meshes/left/Left_hand_palm_link.STL scale=1 1 1
- link base_link: mass 0.15 -> None; geometry collision mesh filename=../mjcf/collision_meshes/left_base_link.stl; visual mesh filename=../meshes/left/base_link.STL scale=1 1 1
- link left_hand_index_DIP_link: mass 0.015 -> None; geometry collision mesh filename=../mjcf/collision_meshes/left_left_hand_index_DIP_link.stl; visual mesh filename=../meshes/left/left_hand_index_DIP_link.STL scale=1 1 1
- link left_hand_index_MCP_link: mass 0.03 -> None; geometry collision mesh filename=../mjcf/collision_meshes/left_left_hand_index_MCP_link.stl; visual mesh filename=../meshes/left/left_hand_index_MCP_link.STL scale=1 1 1
- link left_hand_index_PIP_link: mass 0.04 -> None; geometry collision mesh filename=../mjcf/collision_meshes/left_left_hand_index_PIP_link.stl; visual mesh filename=../meshes/left/left_hand_index_PIP_link.STL scale=1 1 1
- link left_hand_index_swing_link: mass 0.07 -> None; geometry collision mesh filename=../mjcf/collision_meshes/left_left_hand_index_swing_link.stl; visual mesh filename=../meshes/left/left_hand_index_swing_link.STL scale=1 1 1
- link left_hand_mid_DIP_link: mass 0.015 -> None; geometry collision mesh filename=../mjcf/collision_meshes/left_left_hand_mid_DIP_link.stl; visual mesh filename=../meshes/left/left_hand_mid_DIP_link.STL scale=1 1 1
- link left_hand_mid_MCP_link: mass 0.03 -> None; geometry collision mesh filename=../mjcf/collision_meshes/left_left_hand_mid_MCP_link.stl; visual mesh filename=../meshes/left/left_hand_mid_MCP_link.STL scale=1 1 1
- link left_hand_mid_PIP_link: mass 0.04 -> None; geometry collision mesh filename=../mjcf/collision_meshes/left_left_hand_mid_PIP_link.stl; visual mesh filename=../meshes/left/left_hand_mid_PIP_link.STL scale=1 1 1
- link left_hand_mid_swing_link: mass 0.07 -> None; geometry collision mesh filename=../mjcf/collision_meshes/left_left_hand_mid_swing_link.stl; visual mesh filename=../meshes/left/left_hand_mid_swing_link.STL scale=1 1 1
- link left_hand_pinky_DIP_link: mass 0.015 -> None; geometry collision mesh filename=../mjcf/collision_meshes/left_left_hand_pinky_DIP_link.stl; visual mesh filename=../meshes/left/left_hand_pinky_DIP_link.STL scale=1 1 1
- link left_hand_pinky_MCP_link: mass 0.03 -> None; geometry collision mesh filename=../mjcf/collision_meshes/left_left_hand_pinky_MCP_link.stl; visual mesh filename=../meshes/left/left_hand_pinky_MCP_link.STL scale=1 1 1
- link left_hand_pinky_PIP_link: mass 0.04 -> None; geometry collision mesh filename=../mjcf/collision_meshes/left_left_hand_pinky_PIP_link.stl; visual mesh filename=../meshes/left/left_hand_pinky_PIP_link.STL scale=1 1 1
- link left_hand_pinky_swing_link: mass 0.07 -> None; geometry collision mesh filename=../mjcf/collision_meshes/left_left_hand_pinky_swing_link.stl; visual mesh filename=../meshes/left/left_hand_pinky_swing_link.STL scale=1 1 1
- link left_hand_ring_DIP_link: mass 0.015 -> None; geometry collision mesh filename=../mjcf/collision_meshes/left_left_hand_ring_DIP_link.stl; visual mesh filename=../meshes/left/left_hand_ring_DIP_link.STL scale=1 1 1
- link left_hand_ring_MCP_link: mass 0.03 -> None; geometry collision mesh filename=../mjcf/collision_meshes/left_left_hand_ring_MCP_link.stl; visual mesh filename=../meshes/left/left_hand_ring_MCP_link.STL scale=1 1 1
- link left_hand_ring_PIP_link: mass 0.04 -> None; geometry collision mesh filename=../mjcf/collision_meshes/left_left_hand_ring_PIP_link.stl; visual mesh filename=../meshes/left/left_hand_ring_PIP_link.STL scale=1 1 1
- link left_hand_ring_swing_link: mass 0.07 -> None; geometry collision mesh filename=../mjcf/collision_meshes/left_left_hand_ring_swing_link.stl; visual mesh filename=../meshes/left/left_hand_ring_swing_link.STL scale=1 1 1
- link left_hand_thumb_MCP_link: mass 0.04 -> None; geometry collision mesh filename=../mjcf/collision_meshes/left_left_hand_thumb_MCP_link.stl; visual mesh filename=../meshes/left/left_hand_thumb_MCP_link.STL scale=1 1 1
- link left_hand_thumb_PIP_link: mass 0.015 -> None; geometry collision mesh filename=../mjcf/collision_meshes/left_left_hand_thumb_PIP_link.stl; visual mesh filename=../meshes/left/left_hand_thumb_PIP_link.STL scale=1 1 1
- link left_hand_thumb_rota_block_link: mass 0.035 -> None; geometry collision mesh filename=../mjcf/collision_meshes/left_left_hand_thumb_rota_block_li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; visual mesh filename=../meshes/left/left_hand_thumb_rota_block_link.STL scale=1 1 1
- link left_hand_thumb_rotaback_link2: mass 0.075 -> None; geometry collision mesh filename=../mjcf/collision_meshes/left_left_hand_thumb_rotaback_link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; visual mesh filename=../meshes/left/left_hand_thumb_rotaback_link2.STL scale=1 1 1
Joints:
- joint left_hand_index_DIP_joint: axis -0.0071426 0.99997 0 -> 0 0 1; limit lower=0.005 upper=1.565 effort=0 velocity=0 -> lower=0.005 upper=1.565 effort=1.0 velocity=1.0; origin xyz=-0.0045 -1.7143E-05 0.026 rpy=0 0 0.0071427 -> xyz=-0.0053114137261469213 0.025846448194837987 -0.0045110466755889644 rpy=-2.7755575615628914e-17 0 0.12903783821920917
- joint left_hand_index_MCP_joint: axis 0.0071426 0.99997 0 -> 0 0 1; limit lower=0.005 upper=1.3 effort=0 velocity=0 -> lower=0.005 upper=1.565 effort=1.0 velocity=1.0; origin xyz=0.02709999999983987 -0.02756999999977609 0.087706999999999702 rpy=0.10917000000000002 0 0 -> xyz=0.027106823283284235 -0.026576387592038783 0.087815835680192231 rpy=1.4508509931644693 0.42625833852372441 3.084615774699254
- joint left_hand_index_PIP_joint: axis 0 1 0 -> 0 0 1; limit lower=0.005 upper=1.565 effort=0 velocity=0 -> lower=0.005 upper=1.565 effort=1.0 velocity=1.0; origin xyz=0.0124998035843944 -7.21403028728883E-05 0.0419999999999996 rpy=0 0 -0.00714266497914731 -> xyz=0.041023546156784746 3.4694469519536142e-18 -0.026999999999999597 rpy=1.5707963267948963 -1.1967399807955119 3.1077098616583827
- joint left_hand_index_swing_joint: axis 0.99997449127694804 -0.0071426042456228696 -0 -> 0 0 1; limit lower=0.0 upper=0.7 effort=0 velocity=0 -> lower=-0.35 upper=0.35 effort=1.0 velocity=1.0; origin xyz=-0.0100997423618902 7.2140302872923E-05 0.0100000000000036 rpy=-0.34999178339007175 0.00244918578392328 -0.00043302698469405154 -> xyz=0.01819644753826806 0.019340354107076171 -0.00099999999999282954 rpy=1.5707963267948957 -0.033882791931409972 2.0005586058915599
- joint left_hand_mid_DIP_joint: axis 0 1 0 -> 0 0 1; limit lower=0.005 upper=1.565 effort=0 velocity=0 -> lower=0.005 upper=1.565 effort=1.0 velocity=1.0; origin xyz=-0.0045 0 0.033 rpy=0 0 0 -> xyz=-0.0053114137261472405 0.025846448194837821 -0.0017315940115265904 rpy=-5.5511151231257827e-17 0 0.12903783821923204
- joint left_hand_mid_MCP_joint: axis 0 1 0 -> 0 0 1; limit lower=0.005 upper=1.3 effort=0 velocity=0 -> lower=0.005 upper=1.565 effort=1.0 velocity=1.0; origin xyz=0.02719999999983987 -0.001499999999776091 0.088137999999999689 rpy=0 0 0 -> xyz=0.02719999953837687 -0.00049999877805580509 0.088138007230611604 rpy=1.5707963267948968 0.4297622790966602 -3.1415926535897896
- joint left_hand_mid_PIP_joint: axis 0 1 0 -> 0 0 1; limit lower=0.005 upper=1.565 effort=0 velocity=0 -> lower=0.005 upper=1.565 effort=1.0 velocity=1.0; origin xyz=0.0124999999999987 0 0.0420000000000107 rpy=0 0 0 -> xyz=0.041023559408067872 2.1684043449710089e-19 -0.026019547123553179 rpy=1.5707963267948974 -1.1967399807954628 -3.1077095759704942
- joint left_hand_mid_swing_joint: axis 1 -0 -0 -> 0 0 1; limit lower=0.0 upper=0.7 effort=0 velocity=0 -> lower=-0.35 upper=0.35 effort=1.0 velocity=1.0; origin xyz=-0.0101000000001837 0 0.0100000000000402 rpy=-0.35000000000000003 0 0 -> xyz=0.017305157670401285 0.018931832119254491 -0.00099998783788761165 rpy=1.570796326794897 0.033883077619299762 2.0005586058915852
- joint left_hand_pinky_DIP_joint: axis 0 1 0 -> 0 0 1; limit lower=0.005 upper=1.565 effort=0 velocity=0 -> lower=0.005 upper=1.565 effort=1.0 velocity=1.0; origin xyz=0 0.00020676 0.026 rpy=0 0 0.025847 -> xyz=-0.0063815055464910009 0.025204810461647131 -0.006034842938728309 rpy=-0.0062711979857275647 0.025075123623853113 -0.00012198116402359176
- joint left_hand_pinky_MCP_joint: axis 0 1 0 -> 0 0 1; limit lower=0.005 upper=1.3 effort=0 velocity=0 -> lower=0.005 upper=1.565 effort=1.0 velocity=1.0; origin xyz=0.027099553596180971 0.04369427660325461 0.070373477949249502 rpy=-0.12149136010481401 -0.0008656534219200207 -0.0070900155149000235 -> xyz=0.0271068232832797 0.044704606014039389 0.070250121398440751 rpy=1.7043559433280713 0.42725082875541354 -3.0931711956586163
- joint left_hand_pinky_PIP_joint: axis 0 1 0 -> 0 0 1; limit lower=0.005 upper=1.565 effort=0 velocity=0 -> lower=0.005 upper=1.565 effort=1.0 velocity=1.0; origin xyz=0.00799999999999894 0 0.0395000000000003 rpy=0 0 0 -> xyz=0.038626320568843936 0 -0.02181000000000018 rpy=1.5707963267948963 -1.3258211702687228 3.0606963287343296
- joint left_hand_pinky_swing_joint: axis 1 -0 -0 -> 0 0 1; limit lower=0.0 upper=0.7 effort=0 velocity=0 -> lower=-0.35 upper=0.35 effort=1.0 velocity=1.0; origin xyz=-0.01079 1.78569661228936E-05 0.0100000000000004 rpy=-0.35000000000000003 0 0 -> xyz=0.018196447538267484 0.019340354107076102 -0.0010000000000004935 rpy=1.5707963267948957 -0.080896324855458834 2.0005586058915581
- joint left_hand_ring_DIP_joint: axis 0 1 0 -> 0 0 1; limit lower=0.005 upper=1.565 effort=0 velocity=0 -> lower=0.005 upper=1.565 effort=1.0 velocity=1.0; origin xyz=-0.0045 2.3612E-05 0.026 rpy=0 0 0 -> xyz=-0.0053114137258253313 0.025846448194971533 -0.0045110466755893131 rpy=-2.7755575615628914e-17 0 0.12903783821922418
- joint left_hand_ring_MCP_joint: axis 0.0071426 0.99997 0 -> 0 0 1; limit lower=0.005 upper=1.3 effort=0 velocity=0 -> lower=0.005 upper=1.565 effort=1.0 velocity=1.0; origin xyz=0.02709999999983987 0.022467000000223909 0.080994999999999706 rpy=-0.087265999999999982 0 0 -> xyz=0.027106823283282962 0.023481417630913871 0.080906629963767754 rpy=1.6667660125609922 0.42864098926106586 -3.1087726476133142
- joint left_hand_ring_PIP_joint: axis 0 1 0 -> 0 0 1; limit lower=0.005 upper=1.565 effort=0 velocity=0 -> lower=0.005 upper=1.565 effort=1.0 velocity=1.0; origin xyz=0.0125 -1.78569661224183E-05 0.0419999999999992 rpy=0 0 0 -> xyz=0.04102354615678494 -1.7347234759768071e-18 -0.026999999999998935 rpy=1.570796326794895 -1.1967399807954981 3.107709861658404
- joint left_hand_ring_swing_joint: axis 1 -0 -0 -> 0 0 1; limit lower=0.0 upper=0.7 effort=0 velocity=0 -> lower=-0.35 upper=0.35 effort=1.0 velocity=1.0; origin xyz=-0.010099614816648 8.99968134946208E-05 0.0100000000000039 rpy=-0.35000000000000003 0 -0.0071426649791471175 -> xyz=0.018196447538267047 0.019340354107075949 -0.00099999999999785677 rpy=1.5707963267948961 -0.03388279193139021 2.0005586058915599
- joint left_hand_thumb_MCP_joint: axis 0 1 0 -> 0 0 1; limit lower=0.005 upper=1.3 effort=0 velocity=0 -> lower=0.005 upper=1.565 effort=1.0 velocity=1.0; origin xyz=0.0144649150176647 -0.00254683238840498 0.051603919362699 rpy=0.111189397663607 -0.0694825965550923 0.556312969281032 -> xyz=0.051777369955726356 -1.3877787807814457e-17 0.0054157007354755024 rpy=0.5275107839615536 -0.9084965891297635 -2.3106248516321068
- joint left_hand_thumb_PIP_joint: axis 0 1 0 -> 0 0 1; limit lower=0.005 upper=1.565 effort=0 velocity=0 -> lower=0.005 upper=1.565 effort=1.0 velocity=1.0; origin xyz=-0.0045 0 0.026 rpy=0 0 0 -> xyz=-0.0053114137218719798 0.025846448194579846 -0.0045110466755894085 rpy=1.6792123247455493e-15 2.4424906541753444e-15 0.12903783821924114
- joint left_hand_thumb_rota_block_joint: limit lower=0 upper=2.09 effort=0 velocity=0 -> lower=0.0 upper=2.09 effort=1.0 velocity=1.0; origin xyz=0.02801636294752307 -0.016556574015771191 0.026543676950453201 rpy=0.23921093766347604 -0.337904402062424 -0.08067354700273463 -> xyz=0.020095209458105473 -0.018319894388608274 0.034425784821471982 rpy=0.409849353962845 0.035990946425296544 -1.099842689237515
- joint left_hand_thumb_rotaback_joint2: axis 1 0 0 -> 0 0 -1; limit lower=0 upper=1.74 effort=0 velocity=0 -> lower=0.0 upper=1.74 effort=1.0 velocity=1.0; origin xyz=-0.00547277582448224 -0.0220067529252978 -0.00192716000000651 rpy=0 0 0 -> xyz=0.025906534761571742 -3.4694469519536142e-18 -0.010516065096279111 rpy=1.5707963267949003 -1.1774916255348222 -0.55582153100282139
