Commit message: Update Ubuntu hand control project and exclude archives

File: assets/hands/TsenseI_hand_v3_2_withid/urdf/TsenseI_hand_right_v3_2_withid.urdf (robot description, URDF)
Before this commit: robot TsenseI_hand_v3_2_withid_right, 22 links, 21 joints
Links:
- link Right_hand_palm_link: mass 0.017 -> None; geometry collision mesh filename=../mjcf/collision_meshes/right_Right_hand_palm_link.stl; visual mesh filename=../meshes/right/Right_hand_palm_link.STL scale=1 1 1
- link base_link: mass 0.15 -> None; geometry collision mesh filename=../mjcf/collision_meshes/right_base_link.stl; visual mesh filename=../meshes/right/base_link.STL scale=1 1 1
- link right_hand_index_DIP_link: mass 0.015 -> None; geometry collision mesh filename=../mjcf/collision_meshes/right_right_hand_index_DIP_link.stl; visual mesh filename=../meshes/right/right_hand_index_DIP_link.STL scale=1 1 1
- link right_hand_index_MCP_link: mass 0.03 -> None; geometry collision mesh filename=../mjcf/collision_meshes/right_right_hand_index_MCP_link.stl; visual mesh filename=../meshes/right/right_hand_index_MCP_link.STL scale=1 1 1
- link right_hand_index_PIP_link: mass 0.04 -> None; geometry collision mesh filename=../mjcf/collision_meshes/right_right_hand_index_PIP_link.stl; visual mesh filename=../meshes/right/right_hand_index_PIP_link.STL scale=1 1 1
- link right_hand_index_swing_link: mass 0.07 -> None; geometry collision mesh filename=../mjcf/collision_meshes/right_right_hand_index_swing_link.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; visual mesh filename=../meshes/right/right_hand_index_swing_link.STL scale=1 1 1
- link right_hand_mid_DIP_link: mass 0.015 -> None; geometry collision mesh filename=../mjcf/collision_meshes/right_right_hand_mid_DIP_link.stl; visual mesh filename=../meshes/right/right_hand_mid_DIP_link.STL scale=1 1 1
- link right_hand_mid_MCP_link: mass 0.03 -> None; geometry collision mesh filename=../mjcf/collision_meshes/right_right_hand_mid_MCP_link.stl; visual mesh filename=../meshes/right/right_hand_mid_MCP_link.STL scale=1 1 1
- link right_hand_mid_PIP_link: mass 0.04 -> None; geometry collision mesh filename=../mjcf/collision_meshes/right_right_hand_mid_PIP_link.stl; visual mesh filename=../meshes/right/right_hand_mid_PIP_link.STL scale=1 1 1
- link right_hand_mid_swing_link: mass 0.07 -> None; geometry collision mesh filename=../mjcf/collision_meshes/right_right_hand_mid_swing_link.stl; visual mesh filename=../meshes/right/right_hand_mid_swing_link.STL scale=1 1 1
- link right_hand_pinky_DIP_link: mass 0.015 -> None; geometry collision mesh filename=../mjcf/collision_meshes/right_right_hand_pinky_DIP_link.stl; visual mesh filename=../meshes/right/right_hand_pinky_DIP_link.STL scale=1 1 1
- link right_hand_pinky_MCP_link: mass 0.03 -> None; geometry collision mesh filename=../mjcf/collision_meshes/right_right_hand_pinky_MCP_link.stl; visual mesh filename=../meshes/right/right_hand_pinky_MCP_link.STL scale=1 1 1
- link right_hand_pinky_PIP_link: mass 0.04 -> None; geometry collision mesh filename=../mjcf/collision_meshes/right_right_hand_pinky_PIP_link.stl; visual mesh filename=../meshes/right/right_hand_pinky_PIP_link.STL scale=1 1 1
- link right_hand_pinky_swing_link: mass 0.07 -> None; geometry collision mesh filename=../mjcf/collision_meshes/right_right_hand_pinky_swing_link.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; visual mesh filename=../meshes/right/right_hand_pinky_swing_link.STL scale=1 1 1
- link right_hand_ring_DIP_link: mass 0.015 -> None; geometry collision mesh filename=../mjcf/collision_meshes/right_right_hand_ring_DIP_link.stl; visual mesh filename=../meshes/right/right_hand_ring_DIP_link.STL scale=1 1 1
- link right_hand_ring_MCP_link: mass 0.03 -> None; geometry collision mesh filename=../mjcf/collision_meshes/right_right_hand_ring_MCP_link.stl; visual mesh filename=../meshes/right/right_hand_ring_MCP_link.STL scale=1 1 1
- link right_hand_ring_PIP_link: mass 0.04 -> None; geometry collision mesh filename=../mjcf/collision_meshes/right_right_hand_ring_PIP_link.stl; visual mesh filename=../meshes/right/right_hand_ring_PIP_link.STL scale=1 1 1
- link right_hand_ring_swing_link: mass 0.07 -> None; geometry collision mesh filename=../mjcf/collision_meshes/right_right_hand_ring_swing_link.s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; visual mesh filename=../meshes/right/right_hand_ring_swing_link.STL scale=1 1 1
- link right_hand_thumb_MCP_link: mass 0.04 -> None; geometry collision mesh filename=../mjcf/collision_meshes/right_right_hand_thumb_MCP_link.stl; visual mesh filename=../meshes/right/right_hand_thumb_MCP_link.STL scale=1 1 1
- link right_hand_thumb_PIP_link: mass 0.015 -> None; geometry collision mesh filename=../mjcf/collision_meshes/right_right_hand_thumb_PIP_link.stl; visual mesh filename=../meshes/right/right_hand_thumb_PIP_link.STL scale=1 1 1
- link right_hand_thumb_rota_block_link: mass 0.035 -> None; geometry collision mesh filename=../mjcf/collision_meshes/right_right_hand_thumb_rota_block_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; visual mesh filename=../meshes/right/right_hand_thumb_rota_block_link.STL scale=1 1 1
- link right_hand_thumb_rotaback_link2: mass 0.075 -> None; geometry collision mesh filename=../mjcf/collision_meshes/right_right_hand_thumb_rotaback_li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; visual mesh filename=../meshes/right/right_hand_thumb_rotaback_link2.STL scale=1 1 1
Joints:
- joint Right_hand_palm_joint: origin xyz=0.023699999999999999 -0.0064999999999999997 0.044138006984399999 rpy=0 0 0 -> xyz=0.0237 -0.0065 0.0441380069844 rpy=0 0 0
- joint right_hand_index_DIP_joint: axis 0.0071425999999999998 0.99997000000000003 0 -> 0 0 -1; limit lower=0.005 upper=1.565 effort=0 velocity=0 -> lower=0.005 upper=1.565 effort=1.0 velocity=1.0; origin xyz=-0.0044999999999999997 1.7142999999999998e-05 0.025999999999999999 rpy=0 0 -0.0071427000000000001 -> xyz=-0.00531141372614692 -0.025846448194838 -0.00451104667558896 rpy=0 0 -0.129037838219209
- joint right_hand_index_MCP_joint: axis -0.0071425999999999998 0.99997000000000003 0 -> 0 0 -1; limit lower=0.005 upper=1.3 effort=0 velocity=0 -> lower=0.005 upper=1.565 effort=1.0 velocity=1.0; origin xyz=0.02709999999983987 0.02756999999977609 0.087706999999999702 rpy=-0.10917000000000003 0 0 -> xyz=0.0271068232832842 0.0265763875920388 0.0878158356801922 rpy=-1.45085099316447 0.426258338523724 -3.08461577469925
- joint right_hand_index_PIP_joint: axis 0 1 0 -> 0 0 -1; limit lower=0.005 upper=1.565 effort=0 velocity=0 -> lower=0.005 upper=1.565 effort=1.0 velocity=1.0; origin xyz=0.012499803584394399 7.2140302872888306e-05 0.0419999999999996 rpy=0 0 0.0071426649791473101 -> xyz=0.0410235461567847 0 -0.0269999999999996 rpy=-1.5707963267949 -1.19673998079551 -3.10770986165838
- joint right_hand_index_swing_joint: axis -0.99997449127694804 -0.0071426042456228696 -0 -> 0 0 -1; limit lower=0.0 upper=0.7 effort=0 velocity=0 -> lower=-0.35 upper=0.35 effort=1.0 velocity=1.0; origin xyz=-0.0100997423618902 -7.2140302872923e-05 0.0100000000000036 rpy=0.34999178339007175 0.00244918578392328 0.00043302698469405154 -> xyz=0.0181964475382681 -0.0193403541070762 -0.00099999999999283 rpy=-1.5707963267949 -0.03388279193141 -2.00055860589156
- joint right_hand_mid_DIP_joint: axis 0 1 0 -> 0 0 -1; limit lower=0.005 upper=1.565 effort=0 velocity=0 -> lower=0.005 upper=1.565 effort=1.0 velocity=1.0; origin xyz=-0.0044999999999999997 0 0.033000000000000002 rpy=0 0 0 -> xyz=-0.00531141372614724 -0.0258464481948378 -0.00173159401152659 rpy=0 0 -0.129037838219232
- joint right_hand_mid_MCP_joint: axis 0 1 0 -> 0 0 -1; limit lower=0.005 upper=1.3 effort=0 velocity=0 -> lower=0.005 upper=1.565 effort=1.0 velocity=1.0; origin xyz=0.02719999999983987 0.001499999999776091 0.088137999999999689 rpy=0 0 0 -> xyz=0.0271999995383769 0.000499998778055805 0.0881380072306116 rpy=-1.5707963267949 0.42976227909666 3.14159265358979
- joint right_hand_mid_PIP_joint: axis 0 1 0 -> 0 0 -1; limit lower=0.005 upper=1.565 effort=0 velocity=0 -> lower=0.005 upper=1.565 effort=1.0 velocity=1.0; origin xyz=0.0124999999999987 0 0.042000000000010702 rpy=0 0 0 -> xyz=0.0410235594080679 0 -0.0260195471235532 rpy=-1.5707963267949 -1.19673998079546 3.10770957597049
- joint right_hand_mid_swing_joint: axis -1 -0 -0 -> 0 0 -1; limit lower=0.0 upper=0.7 effort=0 velocity=0 -> lower=-0.35 upper=0.35 effort=1.0 velocity=1.0; origin xyz=-0.0101000000001837 0 0.010000000000040201 rpy=0.35000000000000003 0 0 -> xyz=0.0173051576704013 -0.0189318321192545 -0.000999987837887612 rpy=-1.5707963267949 0.0338830776192998 -2.00055860589159
- joint right_hand_pinky_DIP_joint: axis 0 1 0 -> 0 0 -1; limit lower=0.005 upper=1.565 effort=0 velocity=0 -> lower=0.005 upper=1.565 effort=1.0 velocity=1.0; origin xyz=0 -0.00020676000000000001 0.025999999999999999 rpy=0 0 -0.025847000000000002 -> xyz=-0.006381505546491 -0.0252048104616471 -0.00603484293872831 rpy=0.00627119798572756 0.0250751236238531 0.000121981164023592
- joint right_hand_pinky_MCP_joint: axis 0 1 0 -> 0 0 -1; limit lower=0.005 upper=1.3 effort=0 velocity=0 -> lower=0.005 upper=1.565 effort=1.0 velocity=1.0; origin xyz=0.027099553596180971 -0.04369427660325461 0.070373477949249502 rpy=0.12149136010481401 -0.00086565342191979866 0.0070900155149000166 -> xyz=0.0271068232832797 -0.0447046060140394 0.0702501213984408 rpy=-1.70435594332807 0.427250828755414 3.09317119565862
- joint right_hand_pinky_PIP_joint: axis 0 1 0 -> 0 0 -1; limit lower=0.005 upper=1.565 effort=0 velocity=0 -> lower=0.005 upper=1.565 effort=1.0 velocity=1.0; origin xyz=0.0079999999999989403 0 0.039500000000000299 rpy=0 0 0 -> xyz=0.0386263205688439 0 -0.0218100000000002 rpy=-1.5707963267949 -1.32582117026872 -3.06069632873433
- joint right_hand_pinky_swing_joint: axis -1 -0 -0 -> 0 0 -1; limit lower=0.0 upper=0.7 effort=0 velocity=0 -> lower=-0.35 upper=0.35 effort=1.0 velocity=1.0; origin xyz=-0.010789999999999999 -1.78569661228936e-05 0.010000000000000399 rpy=0.35000000000000003 0 0 -> xyz=0.0181964475382675 -0.0193403541070761 -0.00100000000000049 rpy=-1.5707963267949 -0.0808963248554588 -2.00055860589156
- joint right_hand_ring_DIP_joint: axis 0 1 0 -> 0 0 -1; limit lower=0.005 upper=1.565 effort=0 velocity=0 -> lower=0.005 upper=1.565 effort=1.0 velocity=1.0; origin xyz=-0.0044999999999999997 -2.3612e-05 0.025999999999999999 rpy=0 0 0 -> xyz=-0.00531141372582533 -0.0258464481949715 -0.00451104667558931 rpy=0 0 -0.129037838219224
- joint right_hand_ring_MCP_joint: axis -0.0071425999999999998 0.99997000000000003 0 -> 0 0 -1; limit lower=0.005 upper=1.3 effort=0 velocity=0 -> lower=0.005 upper=1.565 effort=1.0 velocity=1.0; origin xyz=0.02709999999983987 -0.022467000000223909 0.080994999999999706 rpy=0.087265999999999969 0 0 -> xyz=0.027106823283283 -0.0234814176309139 0.0809066299637678 rpy=-1.66676601256099 0.428640989261066 3.10877264761331
- joint right_hand_ring_PIP_joint: axis 0 1 0 -> 0 0 -1; limit lower=0.005 upper=1.565 effort=0 velocity=0 -> lower=0.005 upper=1.565 effort=1.0 velocity=1.0; origin xyz=0.012500000000000001 1.78569661224183e-05 0.041999999999999198 rpy=0 0 0 -> xyz=0.0410235461567849 0 -0.0269999999999989 rpy=-1.5707963267949 -1.1967399807955 -3.1077098616584
- joint right_hand_ring_swing_joint: axis -1 -0 -0 -> 0 0 -1; limit lower=0.0 upper=0.7 effort=0 velocity=0 -> lower=-0.35 upper=0.35 effort=1.0 velocity=1.0; origin xyz=-0.010099614816648001 -8.9996813494620798e-05 0.0100000000000039 rpy=0.35000000000000003 0 0.0071426649791471175 -> xyz=0.018196447538267 -0.0193403541070759 -0.000999999999997857 rpy=-1.5707963267949 -0.0338827919313902 -2.00055860589156
- joint right_hand_thumb_MCP_joint: axis 0 1 0 -> 0 0 -1; limit lower=0.005 upper=1.3 effort=0 velocity=0 -> lower=0.005 upper=1.565 effort=1.0 velocity=1.0; origin xyz=0.0144649150176647 0.0025468323884049798 0.051603919362699001 rpy=-0.111189397663607 -0.069482596555092258 -0.5563129692810318 -> xyz=0.0517773699557264 0 0.0054157007354755 rpy=-0.527510783961554 -0.908496589129763 2.31062485163211
- joint right_hand_thumb_PIP_joint: axis 0 1 0 -> 0 0 -1; limit lower=0.005 upper=1.565 effort=0 velocity=0 -> lower=0.005 upper=1.565 effort=1.0 velocity=1.0; origin xyz=-0.0044999999999999997 0 0.025999999999999999 rpy=0 0 0 -> xyz=-0.00531141372187198 -0.0258464481945798 -0.00451104667558941 rpy=-1.67921232474555e-15 2.44249065417534e-15 -0.129037838219241
- joint right_hand_thumb_rota_block_joint: limit lower=0 upper=2.09 effort=0 velocity=0 -> lower=0.0 upper=2.09 effort=1.0 velocity=1.0; origin xyz=0.02801636294752307 0.016556574015771191 0.026543676950453201 rpy=-0.23921093766347606 -0.337904402062424 0.080673547002734658 -> xyz=0.0200952094581055 0.0183198943886083 0.034425784821472 rpy=-0.409849353962845 0.0359909464252965 1.09984268923752
- joint right_hand_thumb_rotaback_joint2: axis -1 0 0 -> 0 0 1; limit lower=0 upper=1.74 effort=0 velocity=0 -> lower=0.0 upper=1.74 effort=1.0 velocity=1.0; origin xyz=-0.0054727758244822403 0.022006752925297801 -0.00192716000000651 rpy=0 0 0 -> xyz=0.0259065347615717 0 -0.0105160650962791 rpy=-1.5707963267949 -1.17749162553482 0.555821531002821

Commit message: Update A3.2 joint ranges and opt-in compensation

File: assets/hands/TsenseI_hand_v3_2/urdf/TsenseI_hand_left_v3_2.urdf (robot description, URDF)
Before this commit: robot TsenseI_hand_v3_2_left, 22 links, 21 joints
Joints:
- joint left_hand_index_DIP_joint: limit lower=0.005 upper=1.565 effort=0 velocity=0 -> lower=0.0 upper=1.57 effort=0 velocity=0
- joint left_hand_index_MCP_joint: limit lower=0.005 upper=1.565 effort=0 velocity=0 -> lower=0.0 upper=1.57 effort=0 velocity=0
- joint left_hand_index_PIP_joint: limit lower=0.005 upper=1.565 effort=0 velocity=0 -> lower=0.0 upper=1.57 effort=0 velocity=0
- joint left_hand_mid_DIP_joint: limit lower=0.005 upper=1.565 effort=0 velocity=0 -> lower=0.0 upper=1.57 effort=0 velocity=0
- joint left_hand_mid_MCP_joint: limit lower=0.005 upper=1.565 effort=0 velocity=0 -> lower=0.0 upper=1.57 effort=0 velocity=0
- joint left_hand_mid_PIP_joint: limit lower=0.005 upper=1.565 effort=0 velocity=0 -> lower=0.0 upper=1.57 effort=0 velocity=0
- joint left_hand_pinky_DIP_joint: limit lower=0.005 upper=1.565 effort=0 velocity=0 -> lower=0.0 upper=1.57 effort=0 velocity=0
- joint left_hand_pinky_MCP_joint: limit lower=0.005 upper=1.565 effort=0 velocity=0 -> lower=0.0 upper=1.57 effort=0 velocity=0
- joint left_hand_pinky_PIP_joint: limit lower=0.005 upper=1.565 effort=0 velocity=0 -> lower=0.0 upper=1.57 effort=0 velocity=0
- joint left_hand_ring_DIP_joint: limit lower=0.005 upper=1.565 effort=0 velocity=0 -> lower=0.0 upper=1.57 effort=0 velocity=0
- joint left_hand_ring_MCP_joint: limit lower=0.005 upper=1.565 effort=0 velocity=0 -> lower=0.0 upper=1.57 effort=0 velocity=0
- joint left_hand_ring_PIP_joint: limit lower=0.005 upper=1.565 effort=0 velocity=0 -> lower=0.0 upper=1.57 effort=0 velocity=0
- joint left_hand_thumb_MCP_joint: limit lower=0.005 upper=1.565 effort=0 velocity=0 -> lower=0.0 upper=1.57 effort=0 velocity=0
- joint left_hand_thumb_PIP_joint: limit lower=0.005 upper=1.565 effort=0 velocity=0 -> lower=0.0 upper=1.57 effort=0 velocity=0

File: assets/hands/TsenseI_hand_v3_2/urdf/TsenseI_hand_right_v3_2.urdf (robot description, URDF)
Before this commit: robot TsenseI_hand_v3_2_right, 22 links, 21 joints
Joints:
- joint right_hand_index_DIP_joint: limit lower=0.005 upper=1.565 effort=0 velocity=0 -> lower=0.0 upper=1.57 effort=0 velocity=0
- joint right_hand_index_MCP_joint: limit lower=0.005 upper=1.565 effort=0 velocity=0 -> lower=0.0 upper=1.57 effort=0 velocity=0
- joint right_hand_index_PIP_joint: limit lower=0.005 upper=1.565 effort=0 velocity=0 -> lower=0.0 upper=1.57 effort=0 velocity=0
- joint right_hand_mid_DIP_joint: limit lower=0.005 upper=1.565 effort=0 velocity=0 -> lower=0.0 upper=1.57 effort=0 velocity=0
- joint right_hand_mid_MCP_joint: limit lower=0.005 upper=1.565 effort=0 velocity=0 -> lower=0.0 upper=1.57 effort=0 velocity=0
- joint right_hand_mid_PIP_joint: limit lower=0.005 upper=1.565 effort=0 velocity=0 -> lower=0.0 upper=1.57 effort=0 velocity=0
- joint right_hand_pinky_DIP_joint: limit lower=0.005 upper=1.565 effort=0 velocity=0 -> lower=0.0 upper=1.57 effort=0 velocity=0
- joint right_hand_pinky_MCP_joint: limit lower=0.005 upper=1.565 effort=0 velocity=0 -> lower=0.0 upper=1.57 effort=0 velocity=0
- joint right_hand_pinky_PIP_joint: limit lower=0.005 upper=1.565 effort=0 velocity=0 -> lower=0.0 upper=1.57 effort=0 velocity=0
- joint right_hand_ring_DIP_joint: limit lower=0.005 upper=1.565 effort=0 velocity=0 -> lower=0.0 upper=1.57 effort=0 velocity=0
- joint right_hand_ring_MCP_joint: limit lower=0.005 upper=1.565 effort=0 velocity=0 -> lower=0.0 upper=1.57 effort=0 velocity=0
- joint right_hand_ring_PIP_joint: limit lower=0.005 upper=1.565 effort=0 velocity=0 -> lower=0.0 upper=1.57 effort=0 velocity=0
- joint right_hand_thumb_MCP_joint: limit lower=0.005 upper=1.565 effort=0 velocity=0 -> lower=0.0 upper=1.57 effort=0 velocity=0
- joint right_hand_thumb_PIP_joint: limit lower=0.005 upper=1.565 effort=0 velocity=0 -> lower=0.0 upper=1.57 effort=0 velocity=0

File: assets/hands/TsenseI_hand_v3_2_withid/urdf/TsenseI_hand_left_v3_2_withid.urdf (robot description, URDF)
Before this commit: robot TsenseI_hand_v3_2_withid_left_raised5mm, 22 links, 21 joints
Joints:
- joint left_hand_index_DIP_joint: limit lower=0.005 upper=1.565 effort=1.0 velocity=1.0 -> lower=0.0 upper=1.57 effort=1.0 velocity=1.0
- joint left_hand_index_MCP_joint: limit lower=0.005 upper=1.565 effort=1.0 velocity=1.0 -> lower=0.0 upper=1.57 effort=1.0 velocity=1.0
- joint left_hand_index_PIP_joint: limit lower=0.005 upper=1.565 effort=1.0 velocity=1.0 -> lower=0.0 upper=1.57 effort=1.0 velocity=1.0
- joint left_hand_mid_DIP_joint: limit lower=0.005 upper=1.565 effort=1.0 velocity=1.0 -> lower=0.0 upper=1.57 effort=1.0 velocity=1.0
- joint left_hand_mid_MCP_joint: limit lower=0.005 upper=1.565 effort=1.0 velocity=1.0 -> lower=0.0 upper=1.57 effort=1.0 velocity=1.0
- joint left_hand_mid_PIP_joint: limit lower=0.005 upper=1.565 effort=1.0 velocity=1.0 -> lower=0.0 upper=1.57 effort=1.0 velocity=1.0
- joint left_hand_pinky_DIP_joint: limit lower=0.005 upper=1.565 effort=1.0 velocity=1.0 -> lower=0.0 upper=1.57 effort=1.0 velocity=1.0
- joint left_hand_pinky_MCP_joint: limit lower=0.005 upper=1.565 effort=1.0 velocity=1.0 -> lower=0.0 upper=1.57 effort=1.0 velocity=1.0
- joint left_hand_pinky_PIP_joint: limit lower=0.005 upper=1.565 effort=1.0 velocity=1.0 -> lower=0.0 upper=1.57 effort=1.0 velocity=1.0
- joint left_hand_ring_DIP_joint: limit lower=0.005 upper=1.565 effort=1.0 velocity=1.0 -> lower=0.0 upper=1.57 effort=1.0 velocity=1.0
- joint left_hand_ring_MCP_joint: limit lower=0.005 upper=1.565 effort=1.0 velocity=1.0 -> lower=0.0 upper=1.57 effort=1.0 velocity=1.0
- joint left_hand_ring_PIP_joint: limit lower=0.005 upper=1.565 effort=1.0 velocity=1.0 -> lower=0.0 upper=1.57 effort=1.0 velocity=1.0
- joint left_hand_thumb_MCP_joint: limit lower=0.005 upper=1.565 effort=1.0 velocity=1.0 -> lower=0.0 upper=1.57 effort=1.0 velocity=1.0
- joint left_hand_thumb_PIP_joint: limit lower=0.005 upper=1.565 effort=1.0 velocity=1.0 -> lower=0.0 upper=1.57 effort=1.0 velocity=1.0

File: assets/hands/TsenseI_hand_v3_2_withid/urdf/TsenseI_hand_right_v3_2_withid.urdf (robot description, URDF)
Before this commit: robot TsenseI_hand_v3_2_withid_right_raised5mm, 22 links, 21 joints
Joints:
- joint right_hand_index_DIP_joint: limit lower=0.005 upper=1.565 effort=1.0 velocity=1.0 -> lower=0.0 upper=1.57 effort=1.0 velocity=1.0
- joint right_hand_index_MCP_joint: limit lower=0.005 upper=1.565 effort=1.0 velocity=1.0 -> lower=0.0 upper=1.57 effort=1.0 velocity=1.0
- joint right_hand_index_PIP_joint: limit lower=0.005 upper=1.565 effort=1.0 velocity=1.0 -> lower=0.0 upper=1.57 effort=1.0 velocity=1.0
- joint right_hand_mid_DIP_joint: limit lower=0.005 upper=1.565 effort=1.0 velocity=1.0 -> lower=0.0 upper=1.57 effort=1.0 velocity=1.0
- joint right_hand_mid_MCP_joint: limit lower=0.005 upper=1.565 effort=1.0 velocity=1.0 -> lower=0.0 upper=1.57 effort=1.0 velocity=1.0
- joint right_hand_mid_PIP_joint: limit lower=0.005 upper=1.565 effort=1.0 velocity=1.0 -> lower=0.0 upper=1.57 effort=1.0 velocity=1.0
- joint right_hand_pinky_DIP_joint: limit lower=0.005 upper=1.565 effort=1.0 velocity=1.0 -> lower=0.0 upper=1.57 effort=1.0 velocity=1.0
- joint right_hand_pinky_MCP_joint: limit lower=0.005 upper=1.565 effort=1.0 velocity=1.0 -> lower=0.0 upper=1.57 effort=1.0 velocity=1.0
- joint right_hand_pinky_PIP_joint: limit lower=0.005 upper=1.565 effort=1.0 velocity=1.0 -> lower=0.0 upper=1.57 effort=1.0 velocity=1.0
- joint right_hand_ring_DIP_joint: limit lower=0.005 upper=1.565 effort=1.0 velocity=1.0 -> lower=0.0 upper=1.57 effort=1.0 velocity=1.0
- joint right_hand_ring_MCP_joint: limit lower=0.005 upper=1.565 effort=1.0 velocity=1.0 -> lower=0.0 upper=1.57 effort=1.0 velocity=1.0
- joint right_hand_ring_PIP_joint: limit lower=0.005 upper=1.565 effort=1.0 velocity=1.0 -> lower=0.0 upper=1.57 effort=1.0 velocity=1.0
- joint right_hand_thumb_MCP_joint: limit lower=0.005 upper=1.565 effort=1.0 velocity=1.0 -> lower=0.0 upper=1.57 effort=1.0 velocity=1.0
- joint right_hand_thumb_PIP_joint: limit lower=0.005 upper=1.565 effort=1.0 velocity=1.0 -> lower=0.0 upper=1.57 effort=1.0 velocity=1.0
